File: Solar_HW/Solar.kicad_pcb (KiCad board)
At the start: 4 copper layers, 143.8 x 80.3 mm, 132 parts, among them P1 CONN_01X02, P10 CONN_01X06, P2 CONN_01X02, P3 CONN_01X02, P4 USB_A, P5 CONN_01X02, P6 CONN_01X02, P7 CONN_01X02, P8 CONN_01X03, P9 CONN_02X03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

Commit message: final board tweaks, new BOM, Final Gerber sent to SEED
Other:
- net class Default: trace_width 1.8288 -> 0.4064
